File: MidiMon/MidiMon.brd (EAGLE design)
At the start: 164.9 x 99.7 mm, 55 parts, among them IC1 PIC18F4520-I/P, IC2 6N138, IC5 7805TV, J1 DIN5, J2 DIN5, J4 2.1MMJACKTHM, X1 ECS-100-18-4X

Commit message: Adjustments to PCB Signed-off-by: goslo <digit99@mailinator.com>
Parts:
- moved J5 19.0 mm to (121.5, 97.0)
- moved J3 16.8 mm to (121.5, 93.9)
- moved JP4 14.6 mm to (126.3, 92.9)
- moved JP5 13.6 mm to (129.1, 92.9)
- moved R10 13.5 mm to (114.7, 96.9), turned to 0 degrees
- moved J7 10.5 mm to (108.0, 97.0)
- moved R9 10.0 mm to (114.7, 93.8), turned to 180 degrees
- moved J6 8.54 mm to (108.0, 94.0)
- moved R13 7.36 mm to (101.3, 97.1), turned to 180 degrees
- moved IC1 5.50 mm to (72.0, 73.8)
- moved VR2 5.22 mm to (72.8, 95.4)
- moved C2 4.75 mm to (93.5, 95.8)
- moved C1 4.71 mm to (78.6, 95.9)
- moved X1 4.57 mm to (85.8, 95.6)
- moved R12 3.25 mm to (100.7, 93.9), turned to 0 degrees
Routing:
- net 5V: track 0.00 -> 206.6 mm
- net N$18: track 0.00 -> 175.4 mm, vias 0 -> 3
- net N$15: track 0.00 -> 97.3 mm, vias 0 -> 1
- net VIN: track 0.00 -> 91.8 mm
- net N$14: track 0.00 -> 73.9 mm
- net N$23: track 0.00 -> 71.7 mm
- net MIDI: track 0.00 -> 67.3 mm
- net A: track 0.00 -> 55.3 mm
- net N$24: track 0.00 -> 39.4 mm
- net N$6: track 0.00 -> 37.3 mm
- net N$10: track 0.00 -> 36.7 mm
- net D4: track 0.00 -> 34.6 mm
- net D1: track 0.00 -> 34.6 mm
- net D0: track 0.00 -> 34.6 mm
- net D7: track 0.00 -> 34.6 mm
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