File: MidiMon/MidiMon.brd (EAGLE design)
At the start: 164.9 x 99.7 mm, 55 parts, among them IC1 PIC18F4520-I/P, IC2 6N138, IC5 7805TV, J1 DIN5, J2 DIN5, J4 2.1MMJACKTHM, X1 ECS-100-18-4X

Commit message: Adjustments made Signed-off-by: goslo <digit99@mailinator.com>
Connections:
- removed net N$8: IC1.7, R9.P$2
- new net N$20: IC1.7, J3.1, R9.P$2
- net 5V: now also R10.P$2, R12.P$2, R13.P$2; no longer J3.1
- net N$18: no longer J5.1, J6.1, J7.1, R10.P$2, R12.P$2, R13.P$2
- net N$29: now also J6.1
- net N$30: now also J5.1
- net N$31: now also J7.1
Routing:
- net N$18: track 175.4 -> 35.5 mm, vias 3 -> 1
- net N$30: track 16.7 -> 92.6 mm
- net 5V: track 206.6 -> 240.9 mm
- net N$20: track 0.00 -> 20.4 mm
- net N$29: track 6.03 -> 15.8 mm
- net N$8: track 8.01 -> 0.00 mm
- net VIN: track 91.8 -> 95.5 mm
- net N$31: track 11.2 -> 14.2 mm
- net N$10: track 36.7 -> 39.3 mm
- net A: track 55.3 -> 53.7 mm
- net N$15: track 97.3 -> 98.9 mm, vias 1 -> 0

Commit message: New Power Sw Signed-off-by: goslo <digit99@mailinator.com>
Parts:
- removed J10, SW1: (no value), SparkFun-Connectors:1X01
- J8: device SparkFun-Connectors:1X01 -> SparkFun-Connectors:1X03
- moved J8 5.30 mm to (4.30, 81.8), turned to 270 degrees
Connections:
- removed net N$13: BAT1.9V, J8.1
- net N$10: now also J8.1; no longer SW1.1
- net PWR+1: now also BAT1.9V, J8.2
Routing:
- net PWR+1: track 0.00 -> 39.9 mm
- net N$13: track 27.2 -> 0.00 mm
- net N$10: track 39.3 -> 40.1 mm
Changed lines of the file:
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@@
 <setting verticaltext="up"/>
 </settings>
-<grid distance="0.2" unitdist="mm" unit="mm" style="lines" multiple="1" display="yes" altdistance="5" altunitdist="mil" altunit="mil"/>
+<grid distance="0.5" unitdist="mm" unit="mm" style="lines" multiple="1" display="yes" altdistance="5" altunitdist="mil" altunit="mil"/>
 <layers>
 <layer number="1" name="Top" color="4" fill="1" visible="yes" active="yes"/>
@@
 <attribute name="PACKAGE" value="HC49/US ECS International" x="-29.74" y="225.18" size="1.778" layer="27" rot="R180" display="off"/>
 </element>
-<element name="J8" library="SparkFun-Connectors" library_urn="urn:adsk.eagle:library:513" package="1X01" package3d_urn="urn:adsk.eagle:package:38028/1" value="" x="4.5" y="76.5" smashed="yes">
-<attribute name="VALUE" x="3.23" y="74.976" size="0.6096" layer="27" font="vector" ratio="20" align="top-left"/>
-</element>
-<element name="SW1" library="SparkFun-Connectors" library_urn="urn:adsk.eagle:library:513" package="1X01" package3d_urn="urn:adsk.eagle:package:38028/1" value="" x="4.5" y="81" smashed="yes">
-<attribute name="NAME" x="6.73" y="80.897" size="0.6096" layer="25" font="vector" ratio="20"/>
-<attribute name="VALUE" x="3.23" y="79.476" size="0.6096" layer="27" font="vector" ratio="20" align="top-left"/>
-</element>
-<element name="J10" library="SparkFun-Connectors" library_urn="urn:adsk.eagle:library:513" package="1X01" package3d_urn="urn:adsk.eagle:package:38028/1" value="" x="4.5" y="85.5" smashed="yes">
-<attribute name="VALUE" x="3.23" y="83.976" size="0.6096" layer="27" font="vector" ratio="20" align="top-left"/>
-</element>
 <element name="H1" library="SparkFun-Hardware" package="STAND-OFF-TIGHT" value="STAND-OFFTIGHT" x="6" y="5" smashed="yes">
 <attribute name="NAME" x="6" y="6.651" size="0.6096" layer="25" font="vector" ratio="20" align="bottom-center"/>
@@
 <element name="H4" library="SparkFun-Hardware" package="STAND-OFF-TIGHT" value="STAND-OFFTIGHT" x="159" y="95" smashed="yes">
 <attribute name="NAME" x="158.5" y="96.651" size="0.6096" layer="25" font="vector" ratio="20" align="bottom-center"/>
+</element>
+<element name="J8" library="SparkFun-Connectors" library_urn="urn:adsk.eagle:library:513" package="1X03" package3d_urn="urn:adsk.eagle:package:38063/1" value="" x="4.3" y="81.8" smashed="yes" rot="R270">
+<attribute name="NAME" x="5.697" y="83.07" size="0.6096" layer="25" font="vector" ratio="20" rot="R270"/>
+<attribute name="VALUE" x="2.268" y="83.07" size="0.6096" layer="27" font="vector" ratio="20" rot="R270"/>
 </element>
 </elements>
@@
 <signal name="PWR+1">
 <contactref element="J4" pad="TIP"/>
+<contactref element="J8" pad="2"/>
+<wire x1="16.07" y1="85.69" x2="13.69" y2="85.69" width="0.508" layer="1"/>
+<wire x1="7.26" y1="79.26" x2="7" y2="79.26" width="0.508" layer="1"/>
+<wire x1="7" y1="79.26" x2="4.3" y2="79.26" width="0.508" layer="1"/>
+<wire x1="13.69" y1="85.69" x2="7.26" y2="79.26" width="0.508" layer="1"/>
+<contactref element="BAT1" pad="9V"/>
+<wire x1="25.33" y1="61.35" x2="7.42" y2="79.26" width="0.508" layer="1"/>
+<wire x1="7.42" y1="79.26" x2="7.26" y2="79.26" width="0.508" layer="1"/>
 </signal>
 <signal name="N$1">
@@
 <contactref element="D7" pad="C"/>
 <contactref element="D5" pad="A"/>
-<contactref element="SW1" pad="1"/>
 <wire x1="22.86" y1="90.424" x2="22.86" y2="89.916" width="0.508" layer="1"/>
 <wire x1="22.86" y1="89.916" x2="22.86" y2="88.9" width="0.508" layer="1"/>
@@
 <wire x1="22.86" y1="88.9" x2="22.59" y2="88.9" width="0.508" layer="1"/>
 <wire x1="25.908" y1="96.52" x2="26.4" y2="96.52" width="0.508" layer="1"/>
-<wire x1="4.572" y1="82.804" x2="4.572" y2="81.28" width="0.508" layer="1"/>
-<wire x1="8.128" y1="86.36" x2="4.572" y2="82.804" width="0.508" layer="1"/>
-<wire x1="8.128" y1="90.424" x2="8.128" y2="86.36" width="0.508" layer="1"/>
-<wire x1="12.7" y1="94.996" x2="8.128" y2="90.424" width="0.508" layer="1"/>
+<wire x1="8.128" y1="90.424" x2="12.7" y2="94.996" width="0.508" layer="1"/>
 <wire x1="17.78" y1="94.996" x2="12.7" y2="94.996" width="0.508" layer="1"/>
 <wire x1="22.86" y1="89.916" x2="17.78" y2="94.996" width="0.508" layer="1"/>
-<wire x1="4.572" y1="81.28" x2="4.5" y2="81" width="0.508" layer="1"/>
-</signal>
-<signal name="N$13">
-<contactref element="BAT1" pad="9V"/>
+<wire x1="8.128" y1="90.424" x2="8.128" y2="83.088" width="0.508" layer="1"/>
 <contactref element="J8" pad="1"/>
-<wire x1="10.16" y1="76.2" x2="4.572" y2="76.2" width="0.508" layer="1"/>
-<wire x1="24.892" y1="61.468" x2="10.16" y2="76.2" width="0.508" layer="1"/>
-<wire x1="4.572" y1="76.2" x2="4.5" y2="76.5" width="0.508" layer="1"/>
-<wire x1="24.892" y1="61.468" x2="25.33" y2="61.35" width="0.508" layer="1"/>
+<wire x1="8.128" y1="83.088" x2="5.588" y2="83.088" width="0.508" layer="1"/>
+<wire x1="5.588" y1="83.088" x2="4.3" y2="81.8" width="0.508" layer="1"/>
 </signal>
 <signal name="N$27">
@@
 <signal name="N$25">
 </signal>
+<signal name="N$8">
+</signal>
 </signals>

Commit message: More adjustments Signed-off-by: goslo <digit99@mailinator.com>
Parts:
- removed JP4, JP5: (no value), SparkFun-Retired:1X02
- added S3: 195-2MST, SamacSys_Parts:DIPS774W56P254L726H790Q4N
- moved VR2 26.1 mm to (59.9, 72.7)
- moved R4 6.67 mm to (143.5, 73.1), turned to 270 degrees
- moved R3 6.36 mm to (140.0, 73.3)
- moved R1 4.00 mm to (147.0, 92.6)
- moved R2 3.50 mm to (143.5, 92.6)
- moved R7 3.50 mm to (139.9, 92.6)
- moved R8 3.50 mm to (136.4, 92.6)
- moved BAT1 0.20 mm to (33.8, 9.15)
- flipped R13 to the bottom
Connections:
- removed net N$11: C7.2, C8.1
- removed net N$16: IC1.4, JP5.1, R7.P$2
- new net N$13: IC1.4, R7.P$2, S3.4
- net GND: now also C7.2, C8.1, S3.1, S3.2; no longer JP4.2, JP5.2
- net N$17: now also S3.3; no longer JP4.1
Routing:
- net N$30: track 92.6 -> 31.4 mm
- net D6: track 34.6 -> 80.0 mm, vias 0 -> 2
- net D5: track 34.6 -> 74.0 mm, vias 0 -> 2
- net N$13: track 0.00 -> 36.2 mm, vias 0 -> 1
- net N$24: track 39.5 -> 11.3 mm
- net N$18: track 35.5 -> 7.53 mm, vias 1 -> 0
- net N$16: track 27.4 -> 0.00 mm
- net 5V: track 240.9 -> 218.3 mm, vias 0 -> 2
- net E: track 29.6 -> 42.6 mm
- net GND: track 0.00 -> 12.4 mm, vias 2 -> 4
- net PWR+1: track 39.9 -> 50.5 mm, vias 0 -> 1
- net N$2: track 26.3 -> 16.5 mm
- net MIDI: track 67.3 -> 76.7 mm
- net D2: track 34.6 -> 43.7 mm, vias 0 -> 2
- net D1: track 34.6 -> 43.7 mm, vias 0 -> 2
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