File: MidiMon/MidiMon.brd (EAGLE design)
At the start: 135.1 x 91.2 mm, 55 parts, among them IC1 PIC18F4520-I/P, IC2 6N138, IC5 7805TV, J1 DIN5, J2 SJ1-3535NG, J4 2.1MMJACKTHM, T1 2N3904, X1 ECS-100-18-4X

Commit message: more changes
Signed-off-by: goslo <digit99@mailinator.com>
Parts:
- R4: value 10k -> 1k
- moved IC2 6.50 mm to (58.7, 77.6)
- moved X1 6.50 mm to (62.7, 67.2)
- moved J8 6.50 mm to (3.30, 65.5)
- moved LED1 6.50 mm to (7.47, 59.5)
- moved BAT1 6.50 mm to (55.8, 17.4)
- moved C1 6.50 mm to (55.5, 67.5)
- moved C10 6.50 mm to (40.0, 69.8)
- moved C11 6.50 mm to (27.4, 68.4)
- moved C2 6.50 mm to (70.3, 67.4)
- moved C5 6.50 mm to (48.0, 68.2)
- moved C7 6.50 mm to (103.9, 66.6)
- moved C8 6.50 mm to (110.7, 66.7)
- moved C9 6.50 mm to (36.5, 65.5)
- moved D1 6.50 mm to (69.6, 77.4)
- moved D5 6.50 mm to (40.8, 81.6)
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Routing:
- net D2: track 211.6 -> 200.9 mm
Other:
- board text added: "MidiBox"
