File: MidiMon/MidiMon.sch (EAGLE design)
At the start: 55 parts, among them IC1 PIC18F4520-I/P, IC2 6N138, IC5 7805TV, J1 DIN5, J2 DIN5, J4 2.1MMJACKTHM, X1 ECS-100-18-4X

Commit message: Adjustments made Signed-off-by: goslo <digit99@mailinator.com>
Connections:
- removed net N$8: IC1.RA5/AN4/~SS/HLVDIN/C2OUT, R9.2
- new net N$20: IC1.RA5/AN4/~SS/HLVDIN/C2OUT, J3.1, R9.2
- net 5V: now also R10.2, R12.2, R13.2; no longer J3.1
- net N$18: no longer J5.1, J6.1, J7.1, R10.2, R12.2, R13.2
- net N$29: now also J6.1
- net N$30: now also J5.1
- net N$31: now also J7.1
Other:
- moved on the sheet: J5, J6, R9

Commit message: New Power Sw Signed-off-by: goslo <digit99@mailinator.com>
Parts:
- removed J10, SW1: (no value), SparkFun-Connectors:CONN_01
- J8: device SparkFun-Connectors:CONN_01 -> SparkFun-Connectors:CONN_03
Connections:
- removed net N$13: BAT1.+, J8.1
- net N$10: now also J8.1; no longer SW1.1
- net PWR+1: now also BAT1.+, J8.2
Changed lines of the file:
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@@
 <setting verticaltext="up"/>
 </settings>
-<grid distance="0.2" unitdist="mm" unit="mm" style="lines" multiple="1" display="no" altdistance="0.01" altunitdist="inch" altunit="inch"/>
+<grid distance="0.1" unitdist="inch" unit="inch" style="lines" multiple="1" display="no" altdistance="0.01" altunitdist="inch" altunit="inch"/>
 <layers>
 <layer number="1" name="Top" color="4" fill="1" visible="no" active="no"/>
@@
 <part name="SUPPLY20" library="supply2" library_urn="urn:adsk.eagle:library:372" deviceset="GND" device=""/>
 <part name="SUPPLY21" library="SparkFun-PowerSymbols" deviceset="5V" device=""/>
-<part name="J8" library="SparkFun-Connectors" library_urn="urn:adsk.eagle:library:513" deviceset="CONN_01" device="" package3d_urn="urn:adsk.eagle:package:38028/1"/>
-<part name="SW1" library="SparkFun-Connectors" library_urn="urn:adsk.eagle:library:513" deviceset="CONN_01" device="" package3d_urn="urn:adsk.eagle:package:38028/1"/>
-<part name="J10" library="SparkFun-Connectors" library_urn="urn:adsk.eagle:library:513" deviceset="CONN_01" device="" package3d_urn="urn:adsk.eagle:package:38028/1"/>
 <part name="H1" library="SparkFun-Hardware" deviceset="STAND-OFF" device="TIGHT"/>
 <part name="H2" library="SparkFun-Hardware" deviceset="STAND-OFF" device="TIGHT"/>
 <part name="H3" library="SparkFun-Hardware" deviceset="STAND-OFF" device="TIGHT"/>
 <part name="H4" library="SparkFun-Hardware" deviceset="STAND-OFF" device="TIGHT"/>
+<part name="J8" library="SparkFun-Connectors" library_urn="urn:adsk.eagle:library:513" deviceset="CONN_03" device="" package3d_urn="urn:adsk.eagle:package:38063/1"/>
 </parts>
 <sheets>
@@
 <attribute name="VALUE" x="16.92" y="113.894" size="1.778" layer="96" align="bottom-center"/>
 </instance>
-<instance part="J8" gate="G$1" x="180.5" y="170.5" smashed="yes" rot="R270">
-<attribute name="VALUE" x="175.674" y="173.04" size="1.778" layer="96" font="vector" rot="R270"/>
-</instance>
-<instance part="SW1" gate="G$1" x="175.52" y="170.4" smashed="yes" rot="R270">
-<attribute name="VALUE" x="170.694" y="172.94" size="1.778" layer="96" font="vector" rot="R270"/>
-<attribute name="NAME" x="173.98" y="173.548" size="1.778" layer="95" font="vector"/>
-</instance>
-<instance part="J10" gate="G$1" x="169.24" y="170.5" smashed="yes" rot="R270">
-<attribute name="VALUE" x="164.414" y="173.04" size="1.778" layer="96" font="vector" rot="R270"/>
-</instance>
 <instance part="H1" gate="G$1" x="-7.62" y="45.72" smashed="yes"/>
 <instance part="H2" gate="G$1" x="-7.62" y="38.1" smashed="yes"/>
 <instance part="H3" gate="G$1" x="0" y="45.72" smashed="yes"/>
 <instance part="H4" gate="G$1" x="0" y="38.1" smashed="yes"/>
+<instance part="J8" gate="J$1" x="177.8" y="175.26" smashed="yes" rot="R270">
+<attribute name="VALUE" x="170.434" y="177.8" size="1.778" layer="96" font="vector" rot="R270"/>
+<attribute name="NAME" x="170.18" y="173.228" size="1.778" layer="95" font="vector"/>
+</instance>
 </instances>
 <busses>
@@
 <net name="PWR+1" class="0">
 <segment>
-<wire x1="200.66" y1="149.86" x2="180.34" y2="149.86" width="0.1524" layer="91"/>
+<wire x1="200.66" y1="149.86" x2="177.8" y2="149.86" width="0.1524" layer="91"/>
 <pinref part="J4" gate="G$1" pin="TIP"/>
+<pinref part="J8" gate="J$1" pin="2"/>
+<wire x1="177.8" y1="167.64" x2="177.8" y2="149.86" width="0.1524" layer="91"/>
+<pinref part="BAT1" gate="G$1" pin="+"/>
+<wire x1="182.88" y1="124.46" x2="177.8" y2="124.46" width="0.1524" layer="91"/>
+<wire x1="177.8" y1="124.46" x2="177.8" y2="149.86" width="0.1524" layer="91"/>
+<junction x="177.8" y="149.86"/>
 </segment>
 </net>
@@
 <wire x1="175" y1="139.7" x2="175" y2="139.5" width="0.1524" layer="91"/>
 <wire x1="175" y1="139.5" x2="175.5" y2="139.5" width="0.1524" layer="91"/>
-<wire x1="175.5" y1="139.5" x2="175.5" y2="157.3" width="0.1524" layer="91"/>
+<wire x1="175.5" y1="139.5" x2="175.5" y2="157.48" width="0.1524" layer="91"/>
 <pinref part="D5" gate="1" pin="A"/>
-<wire x1="175.5" y1="157.3" x2="175.5" y2="157.48" width="0.1524" layer="91"/>
-<wire x1="165.1" y1="157.48" x2="175.5" y2="157.48" width="0.1524" layer="91"/>
-<pinref part="SW1" gate="G$1" pin="1"/>
-<wire x1="175.5" y1="157.48" x2="175.5" y2="162.78" width="0.1524" layer="91"/>
-<wire x1="175.5" y1="162.78" x2="175.52" y2="162.78" width="0.1524" layer="91"/>
-</segment>
-</net>
-<net name="N$13" class="0">
-<segment>
-<pinref part="BAT1" gate="G$1" pin="+"/>
-<wire x1="182.88" y1="124.46" x2="180.5" y2="124.46" width="0.1524" layer="91"/>
-<wire x1="180.5" y1="124.46" x2="180.5" y2="162.88" width="0.1524" layer="91"/>
-<pinref part="J8" gate="G$1" pin="1"/>
-<wire x1="180.5" y1="162.88" x2="180.5" y2="163.38" width="0.1524" layer="91"/>
-<junction x="180.5" y="162.88"/>
+<wire x1="165.1" y1="157.48" x2="175.26" y2="157.48" width="0.1524" layer="91"/>
+<pinref part="J8" gate="J$1" pin="1"/>
+<wire x1="175.26" y1="157.48" x2="175.5" y2="157.48" width="0.1524" layer="91"/>
+<wire x1="175.26" y1="167.64" x2="175.26" y2="157.48" width="0.1524" layer="91"/>
+<junction x="175.26" y="157.48"/>
 </segment>
 </net>
@@
 </segment>
 </net>
+<net name="N$8" class="0">
+<segment>
+<wire x1="175.5" y1="162.78" x2="175.52" y2="162.78" width="0.1524" layer="91"/>
+</segment>
+</net>

Commit message: More adjustments Signed-off-by: goslo <digit99@mailinator.com>
Parts:
- removed JP4, JP5: (no value), SparkFun-Retired:JUMPER-2PTH
- added S3: 195-2MST, SamacSys_Parts:195-2MST
Connections:
- removed net N$11: C7.-, C8.1
- removed net N$16: IC1.RA2/AN2/VREF-/CVREF, JP5.1, R7.2
- new net N$13: IC1.RA2/AN2/VREF-/CVREF, R7.2, S3.4
- net GND: now also C7.-, C8.1, S3.1, S3.2; no longer JP4.2, JP5.2
- net N$17: now also S3.3; no longer JP4.1
Other:
- moved on the sheet: C8
Changed lines of the file:
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@@
 <part name="SUPPLY6" library="supply2" library_urn="urn:adsk.eagle:library:372" deviceset="GND" device=""/>
 <part name="SUPPLY7" library="supply2" library_urn="urn:adsk.eagle:library:372" deviceset="GND" device=""/>
-<part name="JP4" library="SparkFun-Retired" deviceset="JUMPER-2" device="PTH"/>
-<part name="JP5" library="SparkFun-Retired" deviceset="JUMPER-2" device="PTH"/>
 <part name="SUPPLY8" library="supply2" library_urn="urn:adsk.eagle:library:372" deviceset="GND" device=""/>
 <part name="SUPPLY9" library="SparkFun-PowerSymbols" deviceset="5V" device=""/>
@@
 <part name="H4" library="SparkFun-Hardware" deviceset="STAND-OFF" device="TIGHT"/>
 <part name="J8" library="SparkFun-Connectors" library_urn="urn:adsk.eagle:library:513" deviceset="CONN_03" device="" package3d_urn="urn:adsk.eagle:package:38063/1"/>
+<part name="S3" library="SamacSys_Parts" deviceset="195-2MST" device=""/>
 </parts>
 <sheets>
@@
 <attribute name="NAME" x="18.416" y="129.935" size="1.778" layer="95" font="vector"/>
 </instance>
-<instance part="C8" gate="G$1" x="6.9" y="131.5" smashed="yes" rot="R180">
-<attribute name="NAME" x="3.376" y="130.779" size="1.778" layer="95" font="vector" rot="R180"/>
+<instance part="C8" gate="G$1" x="4.36" y="131.5" smashed="yes" rot="R180">
+<attribute name="NAME" x="0.836" y="130.779" size="1.778" layer="95" font="vector" rot="R180"/>
 </instance>
 <instance part="R6" gate="G$1" x="34.66" y="39.08" smashed="yes" rot="R90">
@@
 <instance part="SUPPLY7" gate="GND" x="15.7" y="53.84" smashed="yes">
 <attribute name="VALUE" x="13.795" y="50.665" size="1.778" layer="96"/>
-</instance>
-<instance part="JP4" gate="A" x="-20.5" y="95" smashed="yes" rot="R90">
-<attribute name="NAME" x="-13" y="96.73" size="1.778" layer="95" rot="R180"/>
-<attribute name="VALUE" x="-20.5" y="100.715" size="1.778" layer="96" rot="R180"/>
-</instance>
-<instance part="JP5" gate="A" x="-21" y="100.5" smashed="yes" rot="R90">
-<attribute name="NAME" x="-13.5" y="102.73" size="1.778" layer="95" rot="R180"/>
-<attribute name="VALUE" x="-21" y="106.215" size="1.778" layer="96" rot="R180"/>
 </instance>
 <instance part="SUPPLY8" gate="GND" x="-12.3" y="139.16" smashed="yes">
@@
 <attribute name="VALUE" x="170.434" y="177.8" size="1.778" layer="96" font="vector" rot="R270"/>
 <attribute name="NAME" x="170.18" y="173.228" size="1.778" layer="95" font="vector"/>
+</instance>
+<instance part="S3" gate="G$1" x="-33.02" y="124.46" smashed="yes" rot="R270">
+<attribute name="NAME" x="-25.4" y="107.95" size="1.778" layer="95" rot="R270" align="center-left"/>
 </instance>
 </instances>
@@
 <pinref part="S1" gate="1" pin="P1"/>
 <wire x1="-21.32" y1="122.46" x2="-26" y2="122.46" width="0.1524" layer="91"/>
-<pinref part="JP4" gate="A" pin="2"/>
-<wire x1="-17.96" y1="97.54" x2="-17.96" y2="99" width="0.1524" layer="91"/>
-<wire x1="-17.96" y1="99" x2="-26" y2="99" width="0.1524" layer="91"/>
-<wire x1="-26" y1="99" x2="-26" y2="108.5" width="0.1524" layer="91"/>
-<pinref part="JP5" gate="A" pin="2"/>
-<wire x1="-26" y1="108.5" x2="-26" y2="111.76" width="0.1524" layer="91"/>
-<wire x1="-18.46" y1="103.04" x2="-18.46" y2="108.5" width="0.1524" layer="91"/>
-<wire x1="-18.46" y1="108.5" x2="-26" y2="108.5" width="0.1524" layer="91"/>
-<junction x="-26" y="108.5"/>
 </segment>
 <segment>
@@
 <wire x1="192.46" y1="51.74" x2="192.46" y2="51.08" width="0.1524" layer="91"/>
 </segment>
+<segment>
+<pinref part="S3" gate="G$1" pin="2"/>
+<pinref part="S3" gate="G$1" pin="1"/>
+<wire x1="-35.56" y1="124.46" x2="-33.02" y2="124.46" width="0.1524" layer="91"/>
+<wire x1="-25.8" y1="122.5" x2="-30.6" y2="122.5" width="0.1524" layer="91"/>
+<wire x1="-30.6" y1="122.5" x2="-30.6" y2="124.4" width="0.1524" layer="91"/>
+<wire x1="-30.6" y1="124.4" x2="-33.02" y2="124.4" width="0.1524" layer="91"/>
+<wire x1="-33.02" y1="124.4" x2="-33.02" y2="124.46" width="0.1524" layer="91"/>
+<junction x="-33.02" y="124.46"/>
+</segment>
+<segment>
+<pinref part="C7" gate="G$1" pin="-"/>
+<pinref part="C8" gate="G$1" pin="1"/>
+<wire x1="14.4" y1="126.42" x2="4.36" y2="126.42" width="0.1524" layer="91"/>
+</segment>
 </net>
 <net name="N$4" class="0">
@@
 <pinref part="C8" gate="G$1" pin="2"/>
 <pinref part="C7" gate="G$1" pin="+"/>
-<wire x1="14.4" y1="134.04" x2="6.9" y2="134.04" width="0.1524" layer="91"/>
+<wire x1="14.4" y1="134.04" x2="4.36" y2="134.04" width="0.1524" layer="91"/>
 <wire x1="14.4" y1="134.04" x2="21.4" y2="134" width="0.1524" layer="91"/>
 <junction x="14.4" y="134.04"/>
@@
 </segment>
 </net>
-<net name="N$11" class="0">
-<segment>
-<pinref part="C7" gate="G$1" pin="-"/>
-<pinref part="C8" gate="G$1" pin="1"/>
-<wire x1="14.4" y1="126.42" x2="6.9" y2="126.42" width="0.1524" layer="91"/>
-</segment>
-</net>
 <net name="N$16" class="0">
 <segment>
-<pinref part="IC1" gate="A" pin="RA2/AN2/VREF-/CVREF"/>
-<pinref part="R7" gate="G$1" pin="2"/>
-<wire x1="22.86" y1="99.56" x2="12.62" y2="99.4" width="0.1524" layer="91"/>
-<wire x1="12.66" y1="99.4" x2="12.62" y2="99.4" width="0.1524" layer="91"/>
-<junction x="12.62" y="99.4"/>
-<pinref part="JP5" gate="A" pin="1"/>
-<wire x1="-18.46" y1="100.5" x2="12.62" y2="100.5" width="0.1524" layer="91"/>
-<wire x1="12.62" y1="100.5" x2="12.62" y2="99.4" width="0.1524" layer="91"/>
+<wire x1="-4.4" y1="100.5" x2="-4.4" y2="100.6" width="0.1524" layer="91"/>
 </segment>
 </net>
@@
 <wire x1="12.62" y1="96.78" x2="12.62" y2="96.5" width="0.1524" layer="91"/>
 <junction x="12.62" y="96.78"/>
-<pinref part="JP4" gate="A" pin="1"/>
-<wire x1="12.62" y1="96.78" x2="12.62" y2="95" width="0.1524" layer="91"/>
-<wire x1="12.62" y1="95" x2="-17.96" y2="95" width="0.1524" layer="91"/>
+<wire x1="12.62" y1="96.78" x2="12.62" y2="95.2" width="0.1524" layer="91"/>
+<wire x1="12.62" y1="95.2" x2="-35.5" y2="95.2" width="0.1524" layer="91"/>
+<pinref part="S3" gate="G$1" pin="3"/>
+<wire x1="-35.5" y1="95.2" x2="-35.5" y2="104.14" width="0.1524" layer="91"/>
+<wire x1="-35.5" y1="104.14" x2="-35.56" y2="104.14" width="0.1524" layer="91"/>
 </segment>
 </net>
@@
 </segment>
 </net>
+<net name="N$13" class="0">
+<segment>
+<pinref part="R7" gate="G$1" pin="2"/>
+<pinref part="IC1" gate="A" pin="RA2/AN2/VREF-/CVREF"/>
+<wire x1="22.86" y1="99.56" x2="12.62" y2="99.4" width="0.1524" layer="91"/>
+<wire x1="12.66" y1="99.4" x2="12.62" y2="99.4" width="0.1524" layer="91"/>
+<junction x="12.62" y="99.4"/>
+<wire x1="12.62" y1="99.4" x2="12.62" y2="100.8" width="0.1524" layer="91"/>
+<wire x1="12.62" y1="100.8" x2="12.7" y2="100.8" width="0.1524" layer="91"/>
+<pinref part="S3" gate="G$1" pin="4"/>
+<wire x1="12.62" y1="100.8" x2="-33.02" y2="100.8" width="0.1524" layer="91"/>
+<wire x1="-33.02" y1="100.8" x2="-33.02" y2="104.14" width="0.1524" layer="91"/>
+</segment>
+</net>
+<net name="N$32" class="0">
+<segment>
+<wire x1="-25.9" y1="124.46" x2="-25.9" y2="124.4" width="0.1524" layer="91"/>
+</segment>
+</net>
