File: MidiMon/MidiMon.sch (EAGLE design)
At the start: 55 parts, among them IC1 PIC18F4520-I/P, IC2 6N138, IC5 7805TV, J1 DIN5, J2 SJ1-3535NG, J4 2.1MMJACKTHM, T1 2N3904, X1 ECS-100-18-4X

Commit message: more changes
Signed-off-by: goslo <digit99@mailinator.com>
Parts:
- R4: value 10k -> 1k
Changed lines of the file:
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@@
 <part name="VR2" library="MusicThingModular" deviceset="BOURNS_3362P_TRIMMER" device="P"/>
 <part name="R3" library="SparkFun-Resistors" deviceset="1KOHM" device="-HORIZ-1/4W-5%" value="10k"/>
-<part name="R4" library="SparkFun-Resistors" deviceset="1KOHM" device="-HORIZ-1/4W-5%" value="10k"/>
+<part name="R4" library="SparkFun-Resistors" deviceset="1KOHM" device="-HORIZ-1/4W-5%" value="1k"/>
 <part name="R11" library="SparkFun-Resistors" deviceset="1KOHM" device="-HORIZ-1/4W-5%" value="220"/>
 <part name="D1" library="adafruit" library_urn="urn:adsk.eagle:library:420" deviceset="DIODE" device="DO-1N4148" package3d_urn="urn:adsk.eagle:package:6240748/1"/>
