File: MIn_Core_Display/Min_Core_Display.brd (EAGLE design)
At the start: 103.5 x 48.5 mm, 18 parts, among them U1 SN74HC595D

Commit message: More adjustments Signed-off-by: goslo <digit99@mailinator.com>
Changed lines of the file:
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@@
 <?xml version="1.0" encoding="utf-8"?>
 <!DOCTYPE eagle SYSTEM "eagle.dtd">
-<eagle version="9.2.2">
+<eagle version="9.3.0">
 <drawing>
 <settings>
@@
 </element>
 <element name="R1" library="adafruit" package="R0603" value="1K" x="19.58" y="24.61" smashed="yes">
-<attribute name="NAME" x="20.091" y="28.299" size="0.8128" layer="25"/>
+<attribute name="NAME" x="19.791" y="25.799" size="0.8128" layer="25"/>
 </element>
 <element name="R2" library="adafruit" package="R0603" value="1K" x="19.37" y="21.01" smashed="yes">
