File: Temp/MidiMon_B.sch (EAGLE design)
At the start: 55 parts, among them IC1 PIC18F4520-I/P, IC2 6N138, IC5 7805TV, J1 DIN5, J2 SJ1-3535NG, J4 2.1MMJACKTHM, T1 2N3904, X1 ECS-100-18-4X

Commit message: More changes
Signed-off-by: goslo <digit99@mailinator.com>
Parts:
- removed J2: SJ1-3535NG, SJ1-3535NG:SJ1-3535NG
- removed J9: (no value), SparkFun-Connectors:CONN_02
- removed R14, R15: 220, SparkFun-Resistors:1KOHM-HORIZ-1/4W-5%
- C1, C2: value 33pF -> 18pF
Connections:
- net MIDIIN renamed MIDI
- net PWR renamed PWR+1
- removed net N$21: IC1.RC6/TX/CK, R14.1
- removed net N$33: J9.2, R14.2
- removed net N$34: J9.1, R15.2
- new net N$18: U$2.VDD, VR2.3
- new net N$23: C10.1, C5.+, IC5.VO, R20.1
- net 5V: no longer C10.1, C5.+, IC2.VCC, IC5.VO, R15.1, R20.1, U$2.VDD, VR2.3
- net GND: no longer IC2.GND, J2.1
- net N$5: no longer J2.3
- net N$6: no longer J2.2
