File: MidiMon_v3/MidiMon_v3.brd (EAGLE design)
At the start: 135.1 x 91.2 mm, 55 parts, among them IC1 PIC18F4520-I/P, IC2 6N138, IC5 7805TV, J1 DIN5, J2 SJ1-3535NG, J4 2.1MMJACKTHM, T1 2N3904, X1 ECS-100-18-4X

Commit message: more changes
Signed-off-by: goslo <digit99@mailinator.com>
Parts:
- C1, C2: value 18pF -> 33pF
- R4: value 10k -> 1k
- moved J8 8.23 mm to (3.30, 65.5), turned to 90 degrees
- moved IC2 6.50 mm to (58.7, 77.6)
- moved X1 6.50 mm to (62.7, 67.2)
- moved LED1 6.50 mm to (7.47, 59.5)
- moved BAT1 6.50 mm to (55.8, 17.4)
- moved C1 6.50 mm to (55.5, 67.5)
- moved C10 6.50 mm to (40.0, 69.8)
- moved C11 6.50 mm to (27.4, 68.4)
- moved C2 6.50 mm to (70.3, 67.4)
- moved C5 6.50 mm to (48.0, 68.2)
- moved C7 6.50 mm to (103.9, 66.6)
- moved C8 6.50 mm to (110.7, 66.7)
- moved C9 6.50 mm to (36.5, 65.5)
- moved D1 6.50 mm to (69.6, 77.4)
- moved D5 6.50 mm to (40.8, 81.6)
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Connections:
- removed net N$23: C10.1, C5.+, IC5.3, R20.1
- new net PWR: BAT1.9V, J4.TIP, J8.2
- net 5V: now also C10.1, C5.+, IC2.8, IC5.3, R20.1; no longer BAT1.9V, J4.TIP, J8.2
- net GND: now also IC2.5
Routing:
- net 5V: track 0.00 -> 339.9 mm
- net D2: track 0.00 -> 200.9 mm, vias 0 -> 5
- net N$21: track 0.00 -> 163.5 mm, vias 0 -> 4
- net K: track 0.00 -> 157.7 mm, vias 0 -> 4
- net D7: track 0.00 -> 142.9 mm, vias 0 -> 4
- net D3: track 0.00 -> 136.0 mm, vias 0 -> 3
- net D6: track 0.00 -> 119.2 mm, vias 0 -> 1
- net D5: track 0.00 -> 113.1 mm, vias 0 -> 4
- net D4: track 0.00 -> 106.6 mm, vias 0 -> 6
- net N$17: track 0.00 -> 104.8 mm, vias 0 -> 2
- net N$13: track 0.00 -> 92.6 mm, vias 0 -> 2
- net N$31: track 0.00 -> 91.2 mm, vias 0 -> 1
- net N$20: track 0.00 -> 84.6 mm, vias 0 -> 2
- net N$29: track 0.00 -> 81.9 mm
- net N$30: track 0.00 -> 81.0 mm
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Other:
- board text added: "Apr 2019 V0.3"
- board text added: "MidiBox"
- board text removed: "Apr 2019 V0.2"

Commit message: more changes
Signed-off-by: goslo <digit99@mailinator.com>
Parts:
- C8: device SparkFun-Capacitors:CAP-PTH-SMALL-KIT -> rcl:C025-024X044
- moved BAT1 0.40 mm to (56.2, 17.4)
- flipped J2 to the top
- flipped S3 to the top
Routing:
- net N$17: track 104.8 -> 97.2 mm, vias 2 -> 0
- net N$5: track 52.0 -> 48.2 mm, vias 1 -> 0
- net N$6: track 56.2 -> 52.3 mm, vias 1 -> 0
- net K: track 157.7 -> 159.6 mm
- net D6: track 119.2 -> 118.4 mm
- net N$13: vias 2 -> 1
Other:
- board text added: "May 2019 V0.3"
- board text removed: "Apr 2019 V0.3"
