File: MidiMon_v3/MidiMon_v3.sch (EAGLE design)
At the start: 55 parts, among them IC1 PIC18F4520-I/P, IC2 6N138, IC5 7805TV, J1 DIN5, J2 SJ1-3535NG, J4 2.1MMJACKTHM, T1 2N3904, X1 ECS-100-18-4X

Commit message: more changes
Signed-off-by: goslo <digit99@mailinator.com>
Parts:
- C1, C2: value 18pF -> 33pF
- R4: value 10k -> 1k
Connections:
- net 5V: now also IC2.VCC
- net GND: now also IC2.GND
Changed lines of the file:
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@@
 <setting verticaltext="up"/>
 </settings>
-<grid distance="0.1" unitdist="mm" unit="mm" style="lines" multiple="1" display="no" altdistance="0.01" altunitdist="inch" altunit="inch"/>
+<grid distance="0.1" unitdist="inch" unit="inch" style="lines" multiple="1" display="no" altdistance="0.01" altunitdist="inch" altunit="inch"/>
 <layers>
 <layer number="1" name="Top" color="4" fill="1" visible="no" active="no"/>
@@
 <part name="J1" library="SparkFun-Connectors" library_urn="urn:adsk.eagle:library:513" deviceset="DIN5" device="" package3d_urn="urn:adsk.eagle:package:38294/1"/>
 <part name="X1" library="ECS-100-18-4X" deviceset="ECS-100-18-4X" device=""/>
-<part name="C1" library="SparkFun-Capacitors" deviceset="22PF" device="-PTH-2.54MM-200V-5%" value="18pF"/>
-<part name="C2" library="SparkFun-Capacitors" deviceset="22PF" device="-PTH-2.54MM-200V-5%" value="18pF"/>
+<part name="C1" library="SparkFun-Capacitors" deviceset="22PF" device="-PTH-2.54MM-200V-5%" value="33pF"/>
+<part name="C2" library="SparkFun-Capacitors" deviceset="22PF" device="-PTH-2.54MM-200V-5%" value="33pF"/>
 <part name="C7" library="SparkFun-Capacitors" library_urn="urn:adsk.eagle:library:510" deviceset="10UF-POLAR" device="-RADIAL-2.5MM-25V-20%" package3d_urn="urn:adsk.eagle:package:37423/1" value="10uF"/>
 <part name="C8" library="SparkFun-Capacitors" library_urn="urn:adsk.eagle:library:510" deviceset="0.1UF" device="-KIT-EZ-50V-20%" package3d_urn="urn:adsk.eagle:package:37428/1" value="0.1uF"/>
@@
 <part name="VR2" library="MusicThingModular" deviceset="BOURNS_3362P_TRIMMER" device="P"/>
 <part name="R3" library="SparkFun-Resistors" deviceset="1KOHM" device="-HORIZ-1/4W-5%" value="10k"/>
-<part name="R4" library="SparkFun-Resistors" deviceset="1KOHM" device="-HORIZ-1/4W-5%" value="10k"/>
+<part name="R4" library="SparkFun-Resistors" deviceset="1KOHM" device="-HORIZ-1/4W-5%" value="1k"/>
 <part name="R11" library="SparkFun-Resistors" deviceset="1KOHM" device="-HORIZ-1/4W-5%" value="220"/>
 <part name="D1" library="adafruit" library_urn="urn:adsk.eagle:library:420" deviceset="DIODE" device="DO-1N4148" package3d_urn="urn:adsk.eagle:package:6240748/1"/>
@@
 <part name="SUPPLY2" library="SparkFun-PowerSymbols" deviceset="5V" device=""/>
 <part name="SUPPLY3" library="supply2" library_urn="urn:adsk.eagle:library:372" deviceset="GND" device=""/>
+<part name="SUPPLY18" library="SparkFun-PowerSymbols" deviceset="5V" device=""/>
+<part name="SUPPLY20" library="supply2" library_urn="urn:adsk.eagle:library:372" deviceset="GND" device=""/>
 </parts>
 <sheets>
@@
 <instance part="SUPPLY3" gate="GND" x="117.06" y="20.76" smashed="yes">
 <attribute name="VALUE" x="115.155" y="17.585" size="1.778" layer="96"/>
+</instance>
+<instance part="SUPPLY18" gate="G$1" x="49.9" y="18.76" smashed="yes">
+<attribute name="VALUE" x="49.9" y="21.554" size="1.778" layer="96" align="bottom-center"/>
+</instance>
+<instance part="SUPPLY20" gate="GND" x="39.74" y="44.16" smashed="yes">
+<attribute name="VALUE" x="37.835" y="40.985" size="1.778" layer="96"/>
 </instance>
 </instances>
@@
 <wire x1="117.06" y1="27.94" x2="117.06" y2="23.3" width="0.1524" layer="91"/>
 </segment>
+<segment>
+<pinref part="IC2" gate="G$1" pin="GND"/>
+<pinref part="SUPPLY20" gate="GND" pin="GND"/>
+<wire x1="42.28" y1="39.08" x2="42.28" y2="46.7" width="0.1524" layer="91"/>
+<wire x1="42.28" y1="46.7" x2="39.74" y2="46.7" width="0.1524" layer="91"/>
+</segment>
 </net>
 <net name="N$4" class="0">
@@
 <pinref part="R20" gate="G$1" pin="1"/>
 </segment>
-</net>
+<segment>
+<pinref part="IC2" gate="G$1" pin="VCC"/>
+<pinref part="SUPPLY18" gate="G$1" pin="5V"/>
+<wire x1="42.28" y1="28.92" x2="42.28" y2="18.76" width="0.1524" layer="91"/>
+<wire x1="42.28" y1="18.76" x2="49.9" y2="18.76" width="0.1524" layer="91"/>
+</segment>
+</net>

Commit message: more changes
Signed-off-by: goslo <digit99@mailinator.com>
Parts:
- C8: device SparkFun-Capacitors:0.1UF-KIT-EZ-50V-20% -> rcl:C-EU025-024X044
Changed lines of the file:
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@@
 <part name="C2" library="SparkFun-Capacitors" deviceset="22PF" device="-PTH-2.54MM-200V-5%" value="33pF"/>
 <part name="C7" library="SparkFun-Capacitors" library_urn="urn:adsk.eagle:library:510" deviceset="10UF-POLAR" device="-RADIAL-2.5MM-25V-20%" package3d_urn="urn:adsk.eagle:package:37423/1" value="10uF"/>
-<part name="C8" library="SparkFun-Capacitors" library_urn="urn:adsk.eagle:library:510" deviceset="0.1UF" device="-KIT-EZ-50V-20%" package3d_urn="urn:adsk.eagle:package:37428/1" value="0.1uF"/>
+<part name="C8" library="rcl" library_urn="urn:adsk.eagle:library:334" deviceset="C-EU" device="025-024X044" package3d_urn="urn:adsk.eagle:package:23630/1" value="0.1uF"/>
 <part name="R6" library="SparkFun-Resistors" deviceset="1KOHM" device="-HORIZ-1/4W-5%" value="1.2k"/>
 <part name="R5" library="SparkFun-Resistors" deviceset="1KOHM" device="-HORIZ-1/4W-5%" value="5.6k"/>
@@
 <attribute name="NAME" x="18.416" y="129.935" size="1.778" layer="95" font="vector"/>
 </instance>
-<instance part="C8" gate="G$1" x="4.36" y="131.5" smashed="yes" rot="R180">
-<attribute name="NAME" x="0.836" y="130.779" size="1.778" layer="95" font="vector" rot="R180"/>
+<instance part="C8" gate="G$1" x="4.36" y="128.96" smashed="yes" rot="R180">
+<attribute name="NAME" x="0.836" y="128.239" size="1.778" layer="95" font="vector" rot="R180"/>
 </instance>
 <instance part="R6" gate="G$1" x="34.66" y="39.08" smashed="yes" rot="R90">
@@
 packages will not be understood (or retained) with this version.
 </note>
+<note version="8.4" severity="warning">
+Since Version 8.4, EAGLE supports properties for SPICE simulation.
+Probes in schematics and SPICE mapping objects found in parts and library devices
+will not be understood with this version. Update EAGLE to the latest version
+for full support of SPICE simulation.
+</note>
 </compatibility>
