File: SCS_V2/SCS_V2.brd (EAGLE design)
At the start: 122.8 x 81 mm, 21 parts, among them IC1 74HC165D

Commit message: more changes
Signed-off-by: goslo <digit99@mailinator.com>
Parts:
- moved R4 1.63 mm to (23.1, 2.80)
- moved R9 0.91 mm to (70.4, 16.0), turned to 270 degrees
- moved R2 0.71 mm to (22.1, 11.3)
Routing:
- net VCC: track 0.00 -> 123.4 mm, vias 0 -> 2
- net N$5: track 0.00 -> 101.4 mm, vias 0 -> 1
- net N$3: track 0.00 -> 97.4 mm
- net N$6: track 0.00 -> 72.6 mm, vias 0 -> 1
- net N$9: track 0.00 -> 51.2 mm, vias 0 -> 1
- net N$1: track 0.00 -> 50.7 mm
- net N$7: track 0.00 -> 47.2 mm
- net N$4: track 0.00 -> 46.3 mm, vias 0 -> 1
- net N$2: track 0.00 -> 39.6 mm, vias 0 -> 1
- net N$8: track 0.00 -> 33.7 mm
- net SC: track 0.00 -> 16.0 mm
- net RC: track 0.00 -> 16.0 mm
- net N$11: track 0.00 -> 12.5 mm
Other:
- board size 122.8 x 81 mm -> 122.9 x 81 mm
